File: Keyey/Keyey.kicad_pcb (KiCad board)
At the start: 2 copper layers, 17 parts, among them SW1 Normal, SW2 Caplocks, SW3 Enter, SW4 Tab, SW5 Shift, SW6 Space bar, SW7 Delete

Commit message: July 23-25 update
More info check: https://stardance.hackclub.com/projects/10369
Parts:
- removed A1: RaspberryPi_Pico, Module:RaspberryPi_Pico_Common_SMD
- removed S1: Stab 2u, PCM_Mounting_Keyboard_Stabilizer:Stabilizer_Cherry_MX_2.00u
- removed S2: Stab 6.25u, PCM_marbastlib-mx:STAB_MX_P_6.25u
- removed SW6: Space bar, PCM_marbastlib-mx:SW_MX_1u
- removed SW7: Delete, PCM_marbastlib-mx:SW_MX_1u
- added C10: 100n, Capacitor_SMD:C_0402_1005Metric_Pad0.74x0.62mm_HandSolder, B.Cu at (305.3, -214.4)
- added C100: 0.1uf, Capacitor_SMD:C_01005_0402Metric_Pad0.57x0.30mm_HandSolder, B.Cu at (417.4, -122.4)
- added C101: 0.1uf, Capacitor_SMD:C_01005_0402Metric_Pad0.57x0.30mm_HandSolder, B.Cu at (134.0, -103.3)
- added C102: 0.1uf, Capacitor_SMD:C_01005_0402Metric_Pad0.57x0.30mm_HandSolder, B.Cu at (157.8, -103.1)
- added C103: 0.1uf, Capacitor_SMD:C_01005_0402Metric_Pad0.57x0.30mm_HandSolder, B.Cu at (181.6, -103.2)
- added C104: 0.1uf, Capacitor_SMD:C_01005_0402Metric_Pad0.57x0.30mm_HandSolder, B.Cu at (417.3, -103.3)
- added C105: 0.1uf, Capacitor_SMD:C_01005_0402Metric_Pad0.57x0.30mm_HandSolder, B.Cu at (218.0, -102.3)
- added C106: 0.1uf, Capacitor_SMD:C_01005_0402Metric_Pad0.57x0.30mm_HandSolder, B.Cu at (252.9, -103.1)
- added C107: 0.1uf, Capacitor_SMD:C_01005_0402Metric_Pad0.57x0.30mm_HandSolder, B.Cu at (293.2, -102.3)
- added C108: 0.1uf, Capacitor_SMD:C_01005_0402Metric_Pad0.57x0.30mm_HandSolder, B.Cu at (322.1, -103.2)
- added C109: 0.1uf, Capacitor_SMD:C_01005_0402Metric_Pad0.57x0.30mm_HandSolder, B.Cu at (341.2, -103.2)
- added C11: 100n, Capacitor_SMD:C_0402_1005Metric_Pad0.74x0.62mm_HandSolder, B.Cu at (313.2, -217.3)
- added C110: 0.1uf, Capacitor_SMD:C_01005_0402Metric_Pad0.57x0.30mm_HandSolder, B.Cu at (360.2, -103.1)
- added C111: 0.1uf, Capacitor_SMD:C_01005_0402Metric_Pad0.57x0.30mm_HandSolder, B.Cu at (379.4, -103.2)
- added C112: 0.1uf, Capacitor_SMD:C_01005_0402Metric_Pad0.57x0.30mm_HandSolder, B.Cu at (398.4, -103.3)
- added C113: 0.1uf, Capacitor_SMD:C_01005_0402Metric_Pad0.57x0.30mm_HandSolder, B.Cu at (188.7, -198.4)
- added C12: 100n, Capacitor_SMD:C_0402_1005Metric_Pad0.74x0.62mm_HandSolder, B.Cu at (311.3, -217.3)
- added C13: 100n, Capacitor_SMD:C_0402_1005Metric_Pad0.74x0.62mm_HandSolder, B.Cu at (309.3, -217.3)
- added C14: 100n, Capacitor_SMD:C_0402_1005Metric_Pad0.74x0.62mm_HandSolder, B.Cu at (307.3, -217.3)
- added C15: 100n, Capacitor_SMD:C_0402_1005Metric_Pad0.74x0.62mm_HandSolder, B.Cu at (305.4, -217.3)
- added C16: 100n, Capacitor_SMD:C_0402_1005Metric_Pad0.74x0.62mm_HandSolder, B.Cu at (310.1, -221.8)
- added C17: 4.7u, Capacitor_SMD:C_0402_1005Metric_Pad0.74x0.62mm_HandSolder, B.Cu at (310.1, -219.9)
- added C18: 100n, Capacitor_SMD:C_0402_1005Metric_Pad0.74x0.62mm_HandSolder, B.Cu at (310.1, -223.6)
- added C19: 100n, Capacitor_SMD:C_0402_1005Metric_Pad0.74x0.62mm_HandSolder, B.Cu at (325.2, -219.9)
- added C2: 4.7u, Capacitor_SMD:C_0402_1005Metric_Pad0.74x0.62mm_HandSolder, B.Cu at (288.0, -219.0)
- added C20: 15p, Capacitor_SMD:C_0402_1005Metric_Pad0.74x0.62mm_HandSolder, B.Cu at (285.6, -214.4)
- added C21: 15p, Capacitor_SMD:C_0402_1005Metric_Pad0.74x0.62mm_HandSolder, B.Cu at (289.5, -212.5)
- added C22: 10u, Capacitor_SMD:C_0402_1005Metric_Pad0.74x0.62mm_HandSolder, B.Cu at (313.3, -214.4)
- added C27: 0.1uf, Capacitor_SMD:C_01005_0402Metric_Pad0.57x0.30mm_HandSolder, B.Cu at (131.6, -198.4)
- added C28: 0.1uf, Capacitor_SMD:C_01005_0402Metric_Pad0.57x0.30mm_HandSolder, B.Cu at (150.7, -198.4)
- added C29: 0.1uf, Capacitor_SMD:C_01005_0402Metric_Pad0.57x0.30mm_HandSolder, B.Cu at (169.8, -198.5)
- added C3: 4.7u, Capacitor_SMD:C_0402_1005Metric_Pad0.74x0.62mm_HandSolder, B.Cu at (303.9, -219.0)
- added C32: 0.1uf, Capacitor_SMD:C_01005_0402Metric_Pad0.57x0.30mm_HandSolder, B.Cu at (207.9, -198.8)
- added C33: 0.1uf, Capacitor_SMD:C_01005_0402Metric_Pad0.57x0.30mm_HandSolder, B.Cu at (227.0, -198.7)
- added C34: 0.1uf, Capacitor_SMD:C_01005_0402Metric_Pad0.57x0.30mm_HandSolder, B.Cu at (245.9, -198.7)
- added C35: 0.1uf, Capacitor_SMD:C_01005_0402Metric_Pad0.57x0.30mm_HandSolder, B.Cu at (265.0, -198.7)
- added C36: 0.1uf, Capacitor_SMD:C_01005_0402Metric_Pad0.57x0.30mm_HandSolder, B.Cu at (284.1, -198.7)
- added C37: 0.1uf, Capacitor_SMD:C_01005_0402Metric_Pad0.57x0.30mm_HandSolder, B.Cu at (303.1, -198.8)
- added C38: 0.1uf, Capacitor_SMD:C_01005_0402Metric_Pad0.57x0.30mm_HandSolder, B.Cu at (322.2, -198.7)
- added C39: 0.1uf, Capacitor_SMD:C_01005_0402Metric_Pad0.57x0.30mm_HandSolder, B.Cu at (341.3, -198.5)
- added C4: 4.7u, Capacitor_SMD:C_0402_1005Metric_Pad0.74x0.62mm_HandSolder, B.Cu at (289.1, -220.4)
- added C40: 0.1uf, Capacitor_SMD:C_01005_0402Metric_Pad0.57x0.30mm_HandSolder, B.Cu at (360.3, -198.5)
- added C41: 0.1uf, Capacitor_SMD:C_01005_0402Metric_Pad0.57x0.30mm_HandSolder, B.Cu at (131.6, -179.2)
- added C42: 0.1uf, Capacitor_SMD:C_01005_0402Metric_Pad0.57x0.30mm_HandSolder, B.Cu at (150.7, -179.4)
- added C43: 0.1uf, Capacitor_SMD:C_01005_0402Metric_Pad0.57x0.30mm_HandSolder, B.Cu at (169.8, -179.4)
- added C44: 0.1uf, Capacitor_SMD:C_01005_0402Metric_Pad0.57x0.30mm_HandSolder, B.Cu at (188.8, -179.3)
- added C45: 0.1uf, Capacitor_SMD:C_01005_0402Metric_Pad0.57x0.30mm_HandSolder, B.Cu at (207.8, -179.4)
- added C46: 0.1uf, Capacitor_SMD:C_01005_0402Metric_Pad0.57x0.30mm_HandSolder, B.Cu at (226.9, -179.3)
- added C47: 0.1uf, Capacitor_SMD:C_01005_0402Metric_Pad0.57x0.30mm_HandSolder, B.Cu at (246.0, -179.4)
- added C48: 0.1uf, Capacitor_SMD:C_01005_0402Metric_Pad0.57x0.30mm_HandSolder, B.Cu at (265.0, -179.3)
- added C49: 0.1uf, Capacitor_SMD:C_01005_0402Metric_Pad0.57x0.30mm_HandSolder, B.Cu at (284.1, -179.4)
- added C5: 10u, Capacitor_SMD:C_01005_0402Metric_Pad0.57x0.30mm_HandSolder, B.Cu at (272.1, -215.6)
- added C50: 0.1uf, Capacitor_SMD:C_01005_0402Metric_Pad0.57x0.30mm_HandSolder, B.Cu at (303.2, -179.4)
- added C51: 0.1uf, Capacitor_SMD:C_01005_0402Metric_Pad0.57x0.30mm_HandSolder, B.Cu at (322.1, -179.3)
- added C52: 0.1uf, Capacitor_SMD:C_01005_0402Metric_Pad0.57x0.30mm_HandSolder, B.Cu at (341.2, -179.3)
- added C53: 0.1uf, Capacitor_SMD:C_01005_0402Metric_Pad0.57x0.30mm_HandSolder, B.Cu at (360.3, -179.4)
- added C54: 0.1uf, Capacitor_SMD:C_01005_0402Metric_Pad0.57x0.30mm_HandSolder, B.Cu at (388.7, -179.5)
- added C55: 0.1uf, Capacitor_SMD:C_01005_0402Metric_Pad0.57x0.30mm_HandSolder, B.Cu at (417.3, -179.4)
- added C56: 0.1uf, Capacitor_SMD:C_01005_0402Metric_Pad0.57x0.30mm_HandSolder, B.Cu at (136.4, -160.2)
- added C57: 0.1uf, Capacitor_SMD:C_01005_0402Metric_Pad0.57x0.30mm_HandSolder, B.Cu at (160.2, -160.3)
- added C58: 0.1uf, Capacitor_SMD:C_01005_0402Metric_Pad0.57x0.30mm_HandSolder, B.Cu at (179.2, -160.3)
- added C59: 0.1uf, Capacitor_SMD:C_01005_0402Metric_Pad0.57x0.30mm_HandSolder, B.Cu at (198.2, -160.3)
- added C6: 10u, Capacitor_SMD:C_01005_0402Metric_Pad0.57x0.30mm_HandSolder, B.Cu at (272.1, -220.1)
- added C60: 0.1uf, Capacitor_SMD:C_01005_0402Metric_Pad0.57x0.30mm_HandSolder, B.Cu at (217.3, -160.3)
- added C61: 0.1uf, Capacitor_SMD:C_01005_0402Metric_Pad0.57x0.30mm_HandSolder, B.Cu at (236.3, -160.4)
- added C62: 0.1uf, Capacitor_SMD:C_01005_0402Metric_Pad0.57x0.30mm_HandSolder, B.Cu at (255.3, -160.4)
- added C63: 0.1uf, Capacitor_SMD:C_01005_0402Metric_Pad0.57x0.30mm_HandSolder, B.Cu at (274.5, -160.3)
- added C64: 0.1uf, Capacitor_SMD:C_01005_0402Metric_Pad0.57x0.30mm_HandSolder, B.Cu at (293.5, -160.3)
- added C65: 0.1uf, Capacitor_SMD:C_01005_0402Metric_Pad0.57x0.30mm_HandSolder, B.Cu at (312.6, -160.2)
- added C66: 0.1uf, Capacitor_SMD:C_01005_0402Metric_Pad0.57x0.30mm_HandSolder, B.Cu at (331.6, -160.3)
- added C67: 0.1uf, Capacitor_SMD:C_01005_0402Metric_Pad0.57x0.30mm_HandSolder, B.Cu at (350.7, -160.4)
- added C68: 0.1uf, Capacitor_SMD:C_01005_0402Metric_Pad0.57x0.30mm_HandSolder, B.Cu at (369.7, -160.3)
- added C69: 0.1uf, Capacitor_SMD:C_01005_0402Metric_Pad0.57x0.30mm_HandSolder, B.Cu at (393.6, -160.4)
- added C7: 100n, Capacitor_SMD:C_0402_1005Metric_Pad0.74x0.62mm_HandSolder, B.Cu at (311.2, -214.4)
- added C70: 0.1uf, Capacitor_SMD:C_01005_0402Metric_Pad0.57x0.30mm_HandSolder, B.Cu at (417.4, -160.3)
- added C71: 0.1uf, Capacitor_SMD:C_01005_0402Metric_Pad0.57x0.30mm_HandSolder, B.Cu at (138.8, -141.2)
- added C72: 0.1uf, Capacitor_SMD:C_01005_0402Metric_Pad0.57x0.30mm_HandSolder, B.Cu at (164.9, -141.2)
- added C73: 0.1uf, Capacitor_SMD:C_01005_0402Metric_Pad0.57x0.30mm_HandSolder, B.Cu at (184.0, -141.2)
- added C74: 0.1uf, Capacitor_SMD:C_01005_0402Metric_Pad0.57x0.30mm_HandSolder, B.Cu at (203.0, -141.2)
- added C75: 0.1uf, Capacitor_SMD:C_01005_0402Metric_Pad0.57x0.30mm_HandSolder, B.Cu at (222.1, -141.2)
- added C76: 0.1uf, Capacitor_SMD:C_01005_0402Metric_Pad0.57x0.30mm_HandSolder, B.Cu at (241.0, -141.2)
- added C77: 0.1uf, Capacitor_SMD:C_01005_0402Metric_Pad0.57x0.30mm_HandSolder, B.Cu at (260.2, -141.2)
- added C78: 0.1uf, Capacitor_SMD:C_01005_0402Metric_Pad0.57x0.30mm_HandSolder, B.Cu at (279.3, -141.2)
- added C79: 0.1uf, Capacitor_SMD:C_01005_0402Metric_Pad0.57x0.30mm_HandSolder, B.Cu at (298.3, -141.2)
- added C8: 100n, Capacitor_SMD:C_0402_1005Metric_Pad0.74x0.62mm_HandSolder, B.Cu at (309.3, -214.4)
- added C80: 0.1uf, Capacitor_SMD:C_01005_0402Metric_Pad0.57x0.30mm_HandSolder, B.Cu at (317.4, -141.2)
- added C81: 0.1uf, Capacitor_SMD:C_01005_0402Metric_Pad0.57x0.30mm_HandSolder, B.Cu at (336.4, -141.2)
- added C82: 0.1uf, Capacitor_SMD:C_01005_0402Metric_Pad0.57x0.30mm_HandSolder, B.Cu at (355.4, -141.2)
- added C83: 0.1uf, Capacitor_SMD:C_01005_0402Metric_Pad0.57x0.30mm_HandSolder, B.Cu at (386.4, -141.2)
- added C84: 0.1uf, Capacitor_SMD:C_01005_0402Metric_Pad0.57x0.30mm_HandSolder, B.Cu at (417.3, -141.2)
- added C85: 0.1uf, Capacitor_SMD:C_01005_0402Metric_Pad0.57x0.30mm_HandSolder, B.Cu at (143.6, -122.2)
- added C86: 0.1uf, Capacitor_SMD:C_01005_0402Metric_Pad0.57x0.30mm_HandSolder, B.Cu at (174.5, -122.2)
- added C87: 0.1uf, Capacitor_SMD:C_01005_0402Metric_Pad0.57x0.30mm_HandSolder, B.Cu at (193.4, -122.3)
- added C88: 0.1uf, Capacitor_SMD:C_01005_0402Metric_Pad0.57x0.30mm_HandSolder, B.Cu at (212.6, -122.2)
- added C89: 0.1uf, Capacitor_SMD:C_01005_0402Metric_Pad0.57x0.30mm_HandSolder, B.Cu at (231.6, -122.3)
- added C9: 100n, Capacitor_SMD:C_0402_1005Metric_Pad0.74x0.62mm_HandSolder, B.Cu at (307.3, -214.4)
- added C90: 0.1uf, Capacitor_SMD:C_01005_0402Metric_Pad0.57x0.30mm_HandSolder, B.Cu at (250.7, -122.3)
- added C91: 0.1uf, Capacitor_SMD:C_01005_0402Metric_Pad0.57x0.30mm_HandSolder, B.Cu at (269.7, -122.2)
- added C92: 0.1uf, Capacitor_SMD:C_01005_0402Metric_Pad0.57x0.30mm_HandSolder, B.Cu at (379.2, -198.4)
- added C93: 0.1uf, Capacitor_SMD:C_01005_0402Metric_Pad0.57x0.30mm_HandSolder, B.Cu at (398.3, -198.4)
- added C94: 0.1uf, Capacitor_SMD:C_01005_0402Metric_Pad0.57x0.30mm_HandSolder, B.Cu at (288.8, -122.2)
- added C95: 0.1uf, Capacitor_SMD:C_01005_0402Metric_Pad0.57x0.30mm_HandSolder, B.Cu at (307.8, -122.2)
- added C96: 0.1uf, Capacitor_SMD:C_01005_0402Metric_Pad0.57x0.30mm_HandSolder, B.Cu at (326.8, -122.3)
- added C97: 0.1uf, Capacitor_SMD:C_01005_0402Metric_Pad0.57x0.30mm_HandSolder, B.Cu at (345.9, -122.2)
- added C98: 0.1uf, Capacitor_SMD:C_01005_0402Metric_Pad0.57x0.30mm_HandSolder, B.Cu at (372.2, -122.2)
- added C99: 0.1uf, Capacitor_SMD:C_01005_0402Metric_Pad0.57x0.30mm_HandSolder, B.Cu at (398.4, -122.3)
- added D10: 1N4148W, Diode_SMD:D_SOD-123, B.Cu at (317.9, -199.9)
- added D100: SK6812MINI-E, LED_SMD:LED_SK6812MINI-E_3.2x2.8mm_P1.5mm_ReverseMount, B.Cu at (385.9, -199.9)
- added D101: SK6812MINI-E, LED_SMD:LED_SK6812MINI-E_3.2x2.8mm_P1.5mm_ReverseMount, B.Cu at (404.9, -199.8)
- added D102: SK6812MINI-E, LED_SMD:LED_SK6812MINI-E_3.2x2.8mm_P1.5mm_ReverseMount, B.Cu at (138.3, -180.9)
- added D103: SK6812MINI-E, LED_SMD:LED_SK6812MINI-E_3.2x2.8mm_P1.5mm_ReverseMount, B.Cu at (157.4, -180.9)
- added D104: SK6812MINI-E, LED_SMD:LED_SK6812MINI-E_3.2x2.8mm_P1.5mm_ReverseMount, B.Cu at (176.5, -180.9)
- added D105: SK6812MINI-E, LED_SMD:LED_SK6812MINI-E_3.2x2.8mm_P1.5mm_ReverseMount, B.Cu at (195.5, -180.8)
- added D106: SK6812MINI-E, LED_SMD:LED_SK6812MINI-E_3.2x2.8mm_P1.5mm_ReverseMount, B.Cu at (214.5, -180.8)
- added D107: SK6812MINI-E, LED_SMD:LED_SK6812MINI-E_3.2x2.8mm_P1.5mm_ReverseMount, B.Cu at (233.6, -180.8)
- added D108: SK6812MINI-E, LED_SMD:LED_SK6812MINI-E_3.2x2.8mm_P1.5mm_ReverseMount, B.Cu at (252.6, -180.8)
- added D109: SK6812MINI-E, LED_SMD:LED_SK6812MINI-E_3.2x2.8mm_P1.5mm_ReverseMount, B.Cu at (271.7, -180.8)
- added D11: 1N4148W, Diode_SMD:D_SOD-123, B.Cu at (336.9, -200.1)
- added D110: SK6812MINI-E, LED_SMD:LED_SK6812MINI-E_3.2x2.8mm_P1.5mm_ReverseMount, B.Cu at (290.7, -180.7)
- added D111: SK6812MINI-E, LED_SMD:LED_SK6812MINI-E_3.2x2.8mm_P1.5mm_ReverseMount, B.Cu at (309.9, -180.8)
- added D112: SK6812MINI-E, LED_SMD:LED_SK6812MINI-E_3.2x2.8mm_P1.5mm_ReverseMount, B.Cu at (328.8, -180.8)
- added D113: SK6812MINI-E, LED_SMD:LED_SK6812MINI-E_3.2x2.8mm_P1.5mm_ReverseMount, B.Cu at (347.9, -180.7)
- added D114: SK6812MINI-E, LED_SMD:LED_SK6812MINI-E_3.2x2.8mm_P1.5mm_ReverseMount, B.Cu at (366.9, -180.8)
- added D115: SK6812MINI-E, LED_SMD:LED_SK6812MINI-E_3.2x2.8mm_P1.5mm_ReverseMount, B.Cu at (395.4, -180.8)
- added D116: SK6812MINI-E, LED_SMD:LED_SK6812MINI-E_3.2x2.8mm_P1.5mm_ReverseMount, B.Cu at (424.0, -180.7)
- added D117: SK6812MINI-E, LED_SMD:LED_SK6812MINI-E_3.2x2.8mm_P1.5mm_ReverseMount, B.Cu at (143.0, -161.9)
- added D118: SK6812MINI-E, LED_SMD:LED_SK6812MINI-E_3.2x2.8mm_P1.5mm_ReverseMount, B.Cu at (166.9, -161.8)
- added D119: SK6812MINI-E, LED_SMD:LED_SK6812MINI-E_3.2x2.8mm_P1.5mm_ReverseMount, B.Cu at (185.9, -161.8)
- added D12: 1N4148W, Diode_SMD:D_SOD-123, B.Cu at (356.0, -199.9)
- added D120: SK6812MINI-E, LED_SMD:LED_SK6812MINI-E_3.2x2.8mm_P1.5mm_ReverseMount, B.Cu at (204.8, -161.8)
- added D121: SK6812MINI-E, LED_SMD:LED_SK6812MINI-E_3.2x2.8mm_P1.5mm_ReverseMount, B.Cu at (224.1, -161.9)
- added D122: SK6812MINI-E, LED_SMD:LED_SK6812MINI-E_3.2x2.8mm_P1.5mm_ReverseMount, B.Cu at (242.9, -161.9)
- added D123: SK6812MINI-E, LED_SMD:LED_SK6812MINI-E_3.2x2.8mm_P1.5mm_ReverseMount, B.Cu at (262.0, -161.9)
- added D124: SK6812MINI-E, LED_SMD:LED_SK6812MINI-E_3.2x2.8mm_P1.5mm_ReverseMount, B.Cu at (281.2, -161.9)
- added D125: SK6812MINI-E, LED_SMD:LED_SK6812MINI-E_3.2x2.8mm_P1.5mm_ReverseMount, B.Cu at (300.2, -161.8)
- added D126: SK6812MINI-E, LED_SMD:LED_SK6812MINI-E_3.2x2.8mm_P1.5mm_ReverseMount, B.Cu at (319.3, -162.0)
- added D127: SK6812MINI-E, LED_SMD:LED_SK6812MINI-E_3.2x2.8mm_P1.5mm_ReverseMount, B.Cu at (209.7, -142.8)
- added D128: SK6812MINI-E, LED_SMD:LED_SK6812MINI-E_3.2x2.8mm_P1.5mm_ReverseMount, B.Cu at (424.0, -142.7)
- added D129: SK6812MINI-E, LED_SMD:LED_SK6812MINI-E_3.2x2.8mm_P1.5mm_ReverseMount, B.Cu at (333.6, -123.7)
- added D13: 1N4148W, Diode_SMD:D_SOD-123, B.Cu at (375.0, -199.9)
- added D130: SK6812MINI-E, LED_SMD:LED_SK6812MINI-E_3.2x2.8mm_P1.5mm_ReverseMount, B.Cu at (338.7, -162.0)
- added D131: SK6812MINI-E, LED_SMD:LED_SK6812MINI-E_3.2x2.8mm_P1.5mm_ReverseMount, B.Cu at (228.8, -142.5)
- added D132: SK6812MINI-E, LED_SMD:LED_SK6812MINI-E_3.2x2.8mm_P1.5mm_ReverseMount, B.Cu at (150.2, -123.9)
- added D133: SK6812MINI-E, LED_SMD:LED_SK6812MINI-E_3.2x2.8mm_P1.5mm_ReverseMount, B.Cu at (352.6, -123.7)
- added D134: SK6812MINI-E, LED_SMD:LED_SK6812MINI-E_3.2x2.8mm_P1.5mm_ReverseMount, B.Cu at (357.4, -162.1)
- added D135: SK6812MINI-E, LED_SMD:LED_SK6812MINI-E_3.2x2.8mm_P1.5mm_ReverseMount, B.Cu at (248.1, -142.5)
- added D136: SK6812MINI-E, LED_SMD:LED_SK6812MINI-E_3.2x2.8mm_P1.5mm_ReverseMount, B.Cu at (181.3, -123.9)
- added D137: SK6812MINI-E, LED_SMD:LED_SK6812MINI-E_3.2x2.8mm_P1.5mm_ReverseMount, B.Cu at (379.0, -124.0)
- added D138: SK6812MINI-E, LED_SMD:LED_SK6812MINI-E_3.2x2.8mm_P1.5mm_ReverseMount, B.Cu at (376.7, -162.1)
- added D139: SK6812MINI-E, LED_SMD:LED_SK6812MINI-E_3.2x2.8mm_P1.5mm_ReverseMount, B.Cu at (266.9, -142.5)
- added D14: 1N4148W, Diode_SMD:D_SOD-123, B.Cu at (394.1, -200.0)
- added D140: SK6812MINI-E, LED_SMD:LED_SK6812MINI-E_3.2x2.8mm_P1.5mm_ReverseMount, B.Cu at (238.3, -123.7)
- added D141: SK6812MINI-E, LED_SMD:LED_SK6812MINI-E_3.2x2.8mm_P1.5mm_ReverseMount, B.Cu at (405.1, -123.7)
- added D142: SK6812MINI-E, LED_SMD:LED_SK6812MINI-E_3.2x2.8mm_P1.5mm_ReverseMount, B.Cu at (654.7, -181.4)
- added D143: SK6812MINI-E, LED_SMD:LED_SK6812MINI-E_3.2x2.8mm_P1.5mm_ReverseMount, B.Cu at (286.4, -142.8)
- added D144: SK6812MINI-E, LED_SMD:LED_SK6812MINI-E_3.2x2.8mm_P1.5mm_ReverseMount, B.Cu at (200.2, -124.0)
- added D145: SK6812MINI-E, LED_SMD:LED_SK6812MINI-E_3.2x2.8mm_P1.5mm_ReverseMount, B.Cu at (424.1, -123.9)
- added D146: SK6812MINI-E, LED_SMD:LED_SK6812MINI-E_3.2x2.8mm_P1.5mm_ReverseMount, B.Cu at (400.1, -162.1)
- added D147: SK6812MINI-E, LED_SMD:LED_SK6812MINI-E_3.2x2.8mm_P1.5mm_ReverseMount, B.Cu at (305.1, -142.7)
- added D148: SK6812MINI-E, LED_SMD:LED_SK6812MINI-E_3.2x2.8mm_P1.5mm_ReverseMount, B.Cu at (219.3, -124.0)
- added D149: SK6812MINI-E, LED_SMD:LED_SK6812MINI-E_3.2x2.8mm_P1.5mm_ReverseMount, B.Cu at (235.5, -116.3)
- added D15: 1N4148W, Diode_SMD:D_SOD-123, B.Cu at (413.1, -199.9)
- added D150: SK6812MINI-E, LED_SMD:LED_SK6812MINI-E_3.2x2.8mm_P1.5mm_ReverseMount, B.Cu at (423.9, -162.3)
- added D151: SK6812MINI-E, LED_SMD:LED_SK6812MINI-E_3.2x2.8mm_P1.5mm_ReverseMount, B.Cu at (324.0, -142.8)
- added D152: SK6812MINI-E, LED_SMD:LED_SK6812MINI-E_3.2x2.8mm_P1.5mm_ReverseMount, B.Cu at (257.6, -123.7)
- added D153: SK6812MINI-E, LED_SMD:LED_SK6812MINI-E_3.2x2.8mm_P1.5mm_ReverseMount, B.Cu at (351.0, -88.7)
- added D154: SK6812MINI-E, LED_SMD:LED_SK6812MINI-E_3.2x2.8mm_P1.5mm_ReverseMount, B.Cu at (145.5, -142.8)
- added D155: SK6812MINI-E, LED_SMD:LED_SK6812MINI-E_3.2x2.8mm_P1.5mm_ReverseMount, B.Cu at (343.2, -142.7)
- added D156: SK6812MINI-E, LED_SMD:LED_SK6812MINI-E_3.2x2.8mm_P1.5mm_ReverseMount, B.Cu at (276.4, -123.7)
- added D157: SK6812MINI-E, LED_SMD:LED_SK6812MINI-E_3.2x2.8mm_P1.5mm_ReverseMount, B.Cu at (331.2, -91.7)
- added D158: SK6812MINI-E, LED_SMD:LED_SK6812MINI-E_3.2x2.8mm_P1.5mm_ReverseMount, B.Cu at (171.6, -142.8)
- added D159: SK6812MINI-E, LED_SMD:LED_SK6812MINI-E_3.2x2.8mm_P1.5mm_ReverseMount, B.Cu at (361.9, -142.7)
- added D16: 1N4148W, Diode_SMD:D_SOD-123, B.Cu at (146.4, -180.8)
- added D160: SK6812MINI-E, LED_SMD:LED_SK6812MINI-E_3.2x2.8mm_P1.5mm_ReverseMount, B.Cu at (295.4, -123.7)
- added D161: SK6812MINI-E, LED_SMD:LED_SK6812MINI-E_3.2x2.8mm_P1.5mm_ReverseMount, B.Cu at (164.5, -104.9)
- added D162: SK6812MINI-E, LED_SMD:LED_SK6812MINI-E_3.2x2.8mm_P1.5mm_ReverseMount, B.Cu at (190.7, -142.5)
- added D163: SK6812MINI-E, LED_SMD:LED_SK6812MINI-E_3.2x2.8mm_P1.5mm_ReverseMount, B.Cu at (393.2, -142.7)
- added D164: SK6812MINI-E, LED_SMD:LED_SK6812MINI-E_3.2x2.8mm_P1.5mm_ReverseMount, B.Cu at (314.5, -123.7)
- added D165: SK6812MINI-E, LED_SMD:LED_SK6812MINI-E_3.2x2.8mm_P1.5mm_ReverseMount, B.Cu at (188.2, -104.9)
- added D166: SK6812MINI-E, LED_SMD:LED_SK6812MINI-E_3.2x2.8mm_P1.5mm_ReverseMount, B.Cu at (328.8, -104.9)
- added D167: SK6812MINI-E, LED_SMD:LED_SK6812MINI-E_3.2x2.8mm_P1.5mm_ReverseMount, B.Cu at (347.9, -104.8)
- added D168: SK6812MINI-E, LED_SMD:LED_SK6812MINI-E_3.2x2.8mm_P1.5mm_ReverseMount, B.Cu at (366.9, -104.8)
- added D169: SK6812MINI-E, LED_SMD:LED_SK6812MINI-E_3.2x2.8mm_P1.5mm_ReverseMount, B.Cu at (386.1, -104.8)
- added D17: 1N4148W, Diode_SMD:D_SOD-123, B.Cu at (165.6, -181.0)
- added D170: SK6812MINI-E, LED_SMD:LED_SK6812MINI-E_3.2x2.8mm_P1.5mm_ReverseMount, B.Cu at (405.1, -104.9)
- added D171: SK6812MINI-E, LED_SMD:LED_SK6812MINI-E_3.2x2.8mm_P1.5mm_ReverseMount, B.Cu at (424.0, -104.8)
- added D172: SK6812MINI-E, LED_SMD:LED_SK6812MINI-E_3.2x2.8mm_P1.5mm_ReverseMount, B.Cu at (195.3, -200.2)
- added D18: 1N4148W, Diode_SMD:D_SOD-123, B.Cu at (184.7, -180.9)
- added D19: 1N4148W, Diode_SMD:D_SOD-123, B.Cu at (203.7, -180.9)
- added D20: 1N4148W, Diode_SMD:D_SOD-123, B.Cu at (222.6, -180.9)
- added D21: 1N4148W, Diode_SMD:D_SOD-123, B.Cu at (241.8, -180.9)
- added D22: 1N4148W, Diode_SMD:D_SOD-123, B.Cu at (260.8, -180.9)
- added D23: 1N4148W, Diode_SMD:D_SOD-123, B.Cu at (279.9, -180.9)
- added D24: 1N4148W, Diode_SMD:D_SOD-123, B.Cu at (298.9, -181.0)
- added D25: 1N4148W, Diode_SMD:D_SOD-123, B.Cu at (318.0, -180.9)
- added D26: 1N4148W, Diode_SMD:D_SOD-123, B.Cu at (336.9, -180.8)
- added D27: 1N4148W, Diode_SMD:D_SOD-123, B.Cu at (356.1, -180.9)
- added D28: 1N4148W, Diode_SMD:D_SOD-123, B.Cu at (375.1, -180.9)
- added D29: 1N4148W, Diode_SMD:D_SOD-123, B.Cu at (403.6, -181.0)
- added D30: 1N4148W, Diode_SMD:D_SOD-123, B.Cu at (428.6, -177.4)
- added D31: 1N4148W, Diode_SMD:D_SOD-123, B.Cu at (151.2, -161.8)
- added D32: 1N4148W, Diode_SMD:D_SOD-123, B.Cu at (175.1, -161.9)
- added D33: 1N4148W, Diode_SMD:D_SOD-123, B.Cu at (194.0, -161.8)
- added D34: 1N4148W, Diode_SMD:D_SOD-123, B.Cu at (213.0, -161.9)
- added D35: 1N4148W, Diode_SMD:D_SOD-123, B.Cu at (232.2, -161.9)
- added D36: 1N4148W, Diode_SMD:D_SOD-123, B.Cu at (251.1, -162.0)
- added D37: 1N4148W, Diode_SMD:D_SOD-123, B.Cu at (270.1, -161.9)
- added D38: 1N4148W, Diode_SMD:D_SOD-123, B.Cu at (289.4, -161.8)
- added D39: 1N4148W, Diode_SMD:D_SOD-123, B.Cu at (308.3, -161.8)
- added D40: 1N4148W, Diode_SMD:D_SOD-123, B.Cu at (327.4, -161.8)
- added D41: 1N4148W, Diode_SMD:D_SOD-123, B.Cu at (346.5, -161.9)
- added D42: 1N4148W, Diode_SMD:D_SOD-123, B.Cu at (365.6, -161.9)
- added D43: 1N4148W, Diode_SMD:D_SOD-123, B.Cu at (384.6, -161.9)
- added D44: 1N4148W, Diode_SMD:D_SOD-123, B.Cu at (408.4, -161.9)
- added D45: 1N4148W, Diode_SMD:D_SOD-123, B.Cu at (428.8, -158.3)
- added D46: 1N4148W, Diode_SMD:D_SOD-123, B.Cu at (153.6, -142.7)
- added D47: 1N4148W, Diode_SMD:D_SOD-123, B.Cu at (179.8, -142.8)
- added D48: 1N4148W, Diode_SMD:D_SOD-123, B.Cu at (198.8, -142.7)
- added D49: 1N4148W, Diode_SMD:D_SOD-123, B.Cu at (217.9, -142.7)
- added D50: 1N4148W, Diode_SMD:D_SOD-123, B.Cu at (236.9, -142.8)
- added D51: 1N4148W, Diode_SMD:D_SOD-123, B.Cu at (255.8, -142.8)
- added D52: 1N4148W, Diode_SMD:D_SOD-123, B.Cu at (275.0, -142.8)
- added D53: 1N4148W, Diode_SMD:D_SOD-123, B.Cu at (294.1, -142.7)
- added D54: 1N4148W, Diode_SMD:D_SOD-123, B.Cu at (313.1, -142.8)
- added D55: 1N4148W, Diode_SMD:D_SOD-123, B.Cu at (332.2, -142.8)
- added D56: 1N4148W, Diode_SMD:D_SOD-123, B.Cu at (351.2, -142.7)
- added D57: 1N4148W, Diode_SMD:D_SOD-123, B.Cu at (370.2, -142.7)
- added D58: 1N4148W, Diode_SMD:D_SOD-123, B.Cu at (401.3, -142.7)
- added D59: 1N4148W, Diode_SMD:D_SOD-123, B.Cu at (428.7, -139.2)
- added D60: 1N4148W, Diode_SMD:D_SOD-123, B.Cu at (158.4, -123.8)
- added D61: 1N4148W, Diode_SMD:D_SOD-123, B.Cu at (189.3, -123.8)
- added D62: 1N4148W, Diode_SMD:D_SOD-123, B.Cu at (208.3, -123.8)
- added D63: 1N4148W, Diode_SMD:D_SOD-123, B.Cu at (360.8, -123.7)
- added D64: 1N4148W, Diode_SMD:D_SOD-123, B.Cu at (227.4, -123.8)
- added D65: 1N4148W, Diode_SMD:D_SOD-123, B.Cu at (246.4, -123.8)
- added D66: 1N4148W, Diode_SMD:D_SOD-123, B.Cu at (265.5, -123.8)
- added D67: 1N4148W, Diode_SMD:D_SOD-123, B.Cu at (284.6, -123.8)
- added D68: 1N4148W, Diode_SMD:D_SOD-123, B.Cu at (303.6, -123.8)
- added D69: 1N4148W, Diode_SMD:D_SOD-123, B.Cu at (322.6, -123.8)
- added D70: 1N4148W, Diode_SMD:D_SOD-123, B.Cu at (341.7, -123.9)
- added D71: 1N4148W, Diode_SMD:D_SOD-123, B.Cu at (387.0, -123.8)
- added D72: 1N4148W, Diode_SMD:D_SOD-123, B.Cu at (413.2, -123.8)
- added D73: 1N4148W, Diode_SMD:D_SOD-123, B.Cu at (428.7, -120.4)
- added D74: 1N4148W, Diode_SMD:D_SOD-123, B.Cu at (148.8, -104.8)
- added D75: 1N4148W, Diode_SMD:D_SOD-123, B.Cu at (172.6, -104.7)
- added D76: 1N4148W, Diode_SMD:D_SOD-123, B.Cu at (196.5, -104.8)
- added D77: 1N4148W, Diode_SMD:D_SOD-123, B.Cu at (267.8, -104.6)
- added D78: 1N4148W, Diode_SMD:D_SOD-123, B.Cu at (337.0, -104.7)
- added D79: 1N4148W, Diode_SMD:D_SOD-123, B.Cu at (356.0, -104.7)
- added D8: 1N4148W, Diode_SMD:D_SOD-123, B.Cu at (279.8, -200.0)
- added D80: 1N4148W, Diode_SMD:D_SOD-123, B.Cu at (375.0, -104.7)
- added D81: 1N4148W, Diode_SMD:D_SOD-123, B.Cu at (394.3, -104.8)
- added D82: 1N4148W, Diode_SMD:D_SOD-123, B.Cu at (413.3, -104.9)
- added D83: 1N4148W, Diode_SMD:D_SOD-123, B.Cu at (428.6, -101.3)
- added D84: SK6812MINI-E, LED_SMD:LED_SK6812MINI-E_3.2x2.8mm_P1.5mm_ReverseMount, B.Cu at (138.3, -200.3)
- added D85: SK6812MINI-E, LED_SMD:LED_SK6812MINI-E_3.2x2.8mm_P1.5mm_ReverseMount, B.Cu at (157.3, -200.4)
- added D86: SK6812MINI-E, LED_SMD:LED_SK6812MINI-E_3.2x2.8mm_P1.5mm_ReverseMount, B.Cu at (176.4, -200.4)
- added D87: SK6812MINI-E, LED_SMD:LED_SK6812MINI-E_3.2x2.8mm_P1.5mm_ReverseMount, B.Cu at (214.4, -200.2)
- added D88: SK6812MINI-E, LED_SMD:LED_SK6812MINI-E_3.2x2.8mm_P1.5mm_ReverseMount, B.Cu at (233.7, -200.2)
- added D9: 1N4148W, Diode_SMD:D_SOD-123, B.Cu at (298.8, -200.0)
- added D93: SK6812MINI-E, LED_SMD:LED_SK6812MINI-E_3.2x2.8mm_P1.5mm_ReverseMount, B.Cu at (252.4, -200.0)
- added D94: SK6812MINI-E, LED_SMD:LED_SK6812MINI-E_3.2x2.8mm_P1.5mm_ReverseMount, B.Cu at (271.6, -200.0)
- added D95: SK6812MINI-E, LED_SMD:LED_SK6812MINI-E_3.2x2.8mm_P1.5mm_ReverseMount, B.Cu at (290.6, -200.0)
- added D96: SK6812MINI-E, LED_SMD:LED_SK6812MINI-E_3.2x2.8mm_P1.5mm_ReverseMount, B.Cu at (309.7, -200.0)
- added D97: SK6812MINI-E, LED_SMD:LED_SK6812MINI-E_3.2x2.8mm_P1.5mm_ReverseMount, B.Cu at (328.8, -199.9)
- added D98: SK6812MINI-E, LED_SMD:LED_SK6812MINI-E_3.2x2.8mm_P1.5mm_ReverseMount, B.Cu at (347.9, -199.8)
- added D99: SK6812MINI-E, LED_SMD:LED_SK6812MINI-E_3.2x2.8mm_P1.5mm_ReverseMount, B.Cu at (366.8, -199.9)
- added J1: USB_C_Receptacle_USB2.0_16P, Connector_USB:USB_C_Receptacle_Amphenol_12401948E412A, B.Cu at (281.2, -223.9)
- added J3: Conn_01x03_Pin, Connector_PinHeader_1.00mm:PinHeader_1x03_P1.00mm_Vertical, B.Cu at (258.5, -216.8)
- added L2: AOTA-B201610S3R3-101-T, AOTA-B201610S3R3-101-T:AOTAB201610S3R3101T, B.Cu at (306.3, -222.2)
- added R1: 5.1K, Resistor_SMD:R_01005_0402Metric_Pad0.57x0.30mm_HandSolder, B.Cu at (276.7, -216.6)
- added R10: 1k, Resistor_SMD:R_0402_1005Metric_Pad0.72x0.64mm_HandSolder, B.Cu at (255.6, -219.2)
- added R10close1: 33, Resistor_SMD:R_0402_1005Metric_Pad0.72x0.64mm_HandSolder, B.Cu at (303.2, -221.4)
- added R11: 1k, Resistor_SMD:R_0402_1005Metric_Pad0.72x0.64mm_HandSolder, B.Cu at (288.1, -217.5)
- added R2: 5.1k, Resistor_SMD:R_01005_0402Metric_Pad0.57x0.30mm_HandSolder, B.Cu at (283.8, -216.6)
- added R3: 27, Resistor_SMD:R_0402_1005Metric_Pad0.72x0.64mm_HandSolder, B.Cu at (281.2, -216.2)
- added R4: 27, Resistor_SMD:R_0402_1005Metric_Pad0.72x0.64mm_HandSolder, B.Cu at (279.2, -216.2)
- added SW10: Control, PCM_marbastlib-mx:SW_MX_1u, F.Cu at (140.7, -109.5)
- added SW11: F1, PCM_marbastlib-mx:SW_MX_1u, F.Cu at (157.3, -204.7)
- added SW12: 1, PCM_marbastlib-mx:SW_MX_1u, F.Cu at (157.4, -185.6)
- added SW13: Q, PCM_marbastlib-mx:SW_MX_1u, F.Cu at (166.9, -166.5)
- added SW14: A, PCM_marbastlib-mx:SW_MX_1u, F.Cu at (171.7, -147.4)
- added SW15: Z, PCM_marbastlib-mx:SW_MX_1u, F.Cu at (181.2, -128.4)
- added SW16: Win, PCM_marbastlib-mx:SW_MX_1u, F.Cu at (164.5, -109.3)
- added SW17: F2, PCM_marbastlib-mx:SW_MX_1u, F.Cu at (176.5, -204.7)
- added SW18: 2, PCM_marbastlib-mx:SW_MX_1u, F.Cu at (176.5, -185.5)
- added SW19: W, PCM_marbastlib-mx:SW_MX_1u, F.Cu at (185.9, -166.5)
- added SW20: S, PCM_marbastlib-mx:SW_MX_1u, F.Cu at (190.7, -147.4)
- added SW21: X, PCM_marbastlib-mx:SW_MX_1u, F.Cu at (200.1, -128.5)
- added SW22: F3, PCM_marbastlib-mx:SW_MX_1u, F.Cu at (195.4, -204.7)
- added SW23: 3, PCM_marbastlib-mx:SW_MX_1u, F.Cu at (195.5, -185.6)
- added SW24: E, PCM_marbastlib-mx:SW_MX_1u, F.Cu at (204.9, -166.6)
- added SW25: D, PCM_marbastlib-mx:SW_MX_1u, F.Cu at (209.7, -147.4)
- added SW26: C, PCM_marbastlib-mx:SW_MX_1u, F.Cu at (219.3, -128.4)
- added SW27: F4, PCM_marbastlib-mx:SW_MX_1u, F.Cu at (214.5, -204.7)
- added SW28: 4, PCM_marbastlib-mx:SW_MX_1u, F.Cu at (214.5, -185.6)
- added SW29: R, PCM_marbastlib-mx:SW_MX_1u, F.Cu at (224.0, -166.5)
- added SW30: F, PCM_marbastlib-mx:SW_MX_1u, F.Cu at (228.8, -147.4)
- added SW31: V, PCM_marbastlib-mx:SW_MX_1u, F.Cu at (238.3, -128.5)
- added SW32: opt, PCM_marbastlib-mx:SW_MX_1u, F.Cu at (188.3, -109.4)
- added SW33: F5, PCM_marbastlib-mx:SW_MX_1u, F.Cu at (233.5, -204.7)
- added SW34: 5, PCM_marbastlib-mx:SW_MX_1u, F.Cu at (233.6, -185.6)
- added SW35: T, PCM_marbastlib-mx:SW_MX_1u, F.Cu at (243.0, -166.6)
- added SW36: G, PCM_marbastlib-mx:SW_MX_1u, F.Cu at (247.7, -147.4)
- added SW37: B, PCM_marbastlib-mx:SW_MX_1u, F.Cu at (257.4, -128.5)
- added SW38: F6, PCM_marbastlib-mx:SW_MX_1u, F.Cu at (252.6, -204.6)
- added SW39: 6, PCM_marbastlib-mx:SW_MX_1u, F.Cu at (252.7, -185.6)
- added SW40: Y, PCM_marbastlib-mx:SW_MX_1u, F.Cu at (262.0, -166.6)
- added SW41: H, PCM_marbastlib-mx:SW_MX_1u, F.Cu at (266.9, -147.4)
- added SW42: N, PCM_marbastlib-mx:SW_MX_1u, F.Cu at (276.4, -128.4)
- added SW43: F7, PCM_marbastlib-mx:SW_MX_1u, F.Cu at (271.6, -204.6)
- added SW44: 7, PCM_marbastlib-mx:SW_MX_1u, F.Cu at (271.7, -185.6)
- added SW45: U, PCM_marbastlib-mx:SW_MX_1u, F.Cu at (281.2, -166.5)
- added SW46: J, PCM_marbastlib-mx:SW_MX_1u, F.Cu at (286.0, -147.4)
- added SW47: M, PCM_marbastlib-mx:SW_MX_1u, F.Cu at (295.5, -128.4)
- added SW48: Spacebar, PCM_marbastlib-mx:SW_MX_1u, F.Cu at (259.6, -109.3)
- added SW49: F8, PCM_marbastlib-mx:SW_MX_1u, F.Cu at (290.6, -204.6)
- added SW50: 8, PCM_marbastlib-mx:SW_MX_1u, F.Cu at (290.8, -185.6)
- added SW51: I, PCM_marbastlib-mx:SW_MX_1u, F.Cu at (300.2, -166.5)
- added SW52: K, PCM_marbastlib-mx:SW_MX_1u, F.Cu at (304.9, -147.4)
- added SW53: ,, PCM_marbastlib-mx:SW_MX_1u, F.Cu at (314.5, -128.4)
- added SW54: F9, PCM_marbastlib-mx:SW_MX_1u, F.Cu at (309.7, -204.6)
- added SW55: 9, PCM_marbastlib-mx:SW_MX_1u, F.Cu at (309.9, -185.6)
- added SW56: O, PCM_marbastlib-mx:SW_MX_1u, F.Cu at (319.3, -166.5)
- added SW57: L, PCM_marbastlib-mx:SW_MX_1u, F.Cu at (324.1, -147.4)
- added SW58: ., PCM_marbastlib-mx:SW_MX_1u, F.Cu at (333.5, -128.5)
- added SW59: F10, PCM_marbastlib-mx:SW_MX_1u, F.Cu at (328.8, -204.7)
- added SW60: 0, PCM_marbastlib-mx:SW_MX_1u, F.Cu at (328.8, -185.5)
- added SW61: P, PCM_marbastlib-mx:SW_MX_1u, F.Cu at (338.3, -166.5)
- added SW62: ;, PCM_marbastlib-mx:SW_MX_1u, F.Cu at (343.1, -147.4)
- added SW63: /, PCM_marbastlib-mx:SW_MX_1u, F.Cu at (352.6, -128.4)
- added SW64: F11, PCM_marbastlib-mx:SW_MX_1u, F.Cu at (347.9, -204.6)
- added SW65: -, PCM_marbastlib-mx:SW_MX_1u, F.Cu at (347.9, -185.5)
- added SW66: [, PCM_marbastlib-mx:SW_MX_1u, F.Cu at (357.4, -166.6)
- added SW67: ', PCM_marbastlib-mx:SW_MX_1u, F.Cu at (362.1, -147.4)
- added SW69: F12, PCM_marbastlib-mx:SW_MX_1u, F.Cu at (366.9, -204.6)
- added SW70: =, PCM_marbastlib-mx:SW_MX_1u, F.Cu at (367.0, -185.6)
- added SW71: ], PCM_marbastlib-mx:SW_MX_1u, F.Cu at (376.4, -166.6)
- added SW74: prntsrc, PCM_marbastlib-mx:SW_MX_1u, F.Cu at (385.9, -204.6)
- added SW75: backspace, PCM_marbastlib-mx:SW_MX_1u, F.Cu at (395.4, -185.7)
- added SW76: \, PCM_marbastlib-mx:SW_MX_1u, F.Cu at (400.3, -166.6)
- added SW78: SHIFT, PCM_marbastlib-mx:SW_MX_1u, F.Cu at (378.9, -128.4)
- added SW79: del, PCM_marbastlib-mx:SW_MX_1u, F.Cu at (405.0, -204.6)
- added SW8: Esc, PCM_marbastlib-mx:SW_MX_1u, F.Cu at (138.3, -204.6)
- added SW80: opt, PCM_marbastlib-mx:SW_MX_1u, F.Cu at (328.8, -109.4)
- added SW82: ENTER, PCM_marbastlib-mx:SW_MX_1u, F.Cu at (393.1, -147.4)
- added SW83: up, PCM_marbastlib-mx:SW_MX_1u, F.Cu at (405.1, -128.5)
- added SW84: fn, PCM_marbastlib-mx:SW_MX_1u, F.Cu at (347.9, -109.4)
- added SW85: pgup, PCM_marbastlib-mx:SW_MX_1u, F.Cu at (424.0, -185.6)
- added SW86: pgdn, PCM_marbastlib-mx:SW_MX_1u, F.Cu at (424.1, -166.5)
- added SW87: home, PCM_marbastlib-mx:SW_MX_1u, F.Cu at (424.0, -147.4)
- added SW88: end, PCM_marbastlib-mx:SW_MX_1u, F.Cu at (424.1, -128.6)
- added SW89: Control, PCM_marbastlib-mx:SW_MX_1u, F.Cu at (366.9, -109.3)
- added SW9: ~, PCM_marbastlib-mx:SW_MX_1u, F.Cu at (138.3, -185.5)
- added SW90: left, PCM_marbastlib-mx:SW_MX_1u, F.Cu at (386.1, -109.4)
- added SW91: down, PCM_marbastlib-mx:SW_MX_1u, F.Cu at (405.1, -109.5)
- added SW92: right, PCM_marbastlib-mx:SW_MX_1u, F.Cu at (424.0, -109.5)
- added U2: RP2350B, Package_DFN_QFN:QFN-80-1EP_10x10mm_P0.4mm_EP3.4x3.4mm, B.Cu at (296.9, -218.7)
- added U3: NCP1117-3.3_SOT223, Package_TO_SOT_SMD:SOT-223-3_TabPin2, B.Cu at (266.9, -218.9)
- added U4: W25Q128JVS, Package_SO:SOIC-8_5.3x5.3mm_P1.27mm, B.Cu at (319.5, -221.2)
- added Y1: ABM8-272-T3, ABM8-272-T3:XTAL_ABM8-272-T3, B.Cu at (288.5, -215.0)
- D1, D2, D3, D4, D5, D6, D7: moved to B.Cu
- SW1: value Normal -> EC11E15244G1; footprint PCM_marbastlib-mx:SW_MX_1u -> PCM_marbastlib-various:ROT_Alps_EC11E-Switch
- SW3: value Enter -> SW_Push; footprint PCM_marbastlib-mx:SW_MX_1u -> Button_Switch_SMD:Panasonic_EVQPUJ_EVQPUA; moved to B.Cu
- SW5: value Shift -> Left Shift
- moved SW1 352.5 mm to (423.2, -204.6)
- moved D7 317.1 mm to (260.8, -199.9), turned to 90 degrees
- moved D6 314.6 mm to (241.7, -200.1), turned to 90 degrees
- moved D5 308.9 mm to (222.6, -200.1), turned to 90 degrees
- moved D4 304.2 mm to (203.5, -200.1), turned to 90 degrees
- moved D3 300.8 mm to (184.6, -200.1), turned to 90 degrees
- moved D2 298.4 mm to (165.5, -199.9), turned to 90 degrees
- moved D1 297.5 mm to (146.4, -200.0), turned to 90 degrees
- moved SW3 295.4 mm to (258.3, -222.0), turned to 180 degrees
- moved SW4 260.4 mm to (143.1, -166.5)
- moved SW2 237.7 mm to (145.5, -147.4)
- moved SW5 212.4 mm to (150.3, -128.5)
Connections:
- D1 pad 1: unconnected-(D1-K-Pad1) -> ROW1
- D2 pad 1: unconnected-(D2-K-Pad1) -> ROW1
- D3 pad 1: unconnected-(D3-K-Pad1) -> ROW1
- D4 pad 1: unconnected-(D4-K-Pad1) -> ROW1
- D5 pad 1: unconnected-(D5-K-Pad1) -> ROW1
- D6 pad 1: unconnected-(D6-K-Pad1) -> ROW1
- D7 pad 1: unconnected-(D7-K-Pad1) -> ROW1
- SW2 pad 1: unconnected-(SW2-Pad1) -> COL1
- SW2 pad 2: Net-(D2-A) -> Net-(D46-A)
- SW3 pad 1: unconnected-(SW3-Pad1) -> GND
- SW3 pad 2: Net-(D1-A) -> Net-(R10-Pad2)
- SW4 pad 1: unconnected-(SW4-Pad1) -> COL1
- SW4 pad 2: Net-(D6-A) -> Net-(D31-A)
- SW5 pad 1: unconnected-(SW5-Pad1) -> COL1
- SW5 pad 2: Net-(D3-A) -> Net-(D60-A)
Routing:
- net +5V: track 0.00 -> 1455.6 mm, vias 0 -> 51
- net GND: track 0.00 -> 1350.8 mm, vias 0 -> 4
- net ROW6: track 0.00 -> 437.3 mm, vias 0 -> 2
- net ROW5: track 0.00 -> 401.3 mm, vias 0 -> 2
- net ROW4: track 0.00 -> 383.0 mm, vias 0 -> 2
- net ROW3: track 0.00 -> 375.3 mm, vias 0 -> 2
- net ROW2: track 0.00 -> 341.6 mm, vias 0 -> 2
- net COL1: track 0.00 -> 325.4 mm, vias 0 -> 1
- net Net-(D116-DOUT): track 0.00 -> 316.6 mm, vias 0 -> 2
- net COL2: track 0.00 -> 314.1 mm, vias 0 -> 1
- net ROW1: track 0.00 -> 306.5 mm, vias 0 -> 2
- net COL3: track 0.00 -> 285.3 mm, vias 0 -> 1
- net Net-(D101-DOUT): track 0.00 -> 270.1 mm, vias 0 -> 3
- net COL15: track 0.00 -> 251.6 mm, vias 0 -> 1
- net COL13: track 0.00 -> 238.7 mm, vias 0 -> 1
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Other:
- board outline added: 304.8 x 125.5 mm
- copper layers 2 -> 4
