File: Keyey/Keymatrix.kicad_sch (KiCad schematic)
At the start: 167 parts, among them SW1 EC11E15244G1, SW10 Control, SW11 F1, SW12 1, SW13 Q, SW14 A, SW15 Z, SW16 Win, SW17 F2, SW18 2, SW19 W, SW2 Caplocks, SW20 S, SW21 X, SW22 F3, SW23 3, SW24 E, SW25 D, SW26 C, SW27 F4, SW28 4, SW29 R, SW30 F, SW31 V, SW32 opt, SW33 F5, SW34 5, SW35 T, SW36 G, SW37 B, SW38 F6, SW39 6, SW4 Tab, SW40 Y, SW41 H, SW42 N, SW43 F7, SW44 7, SW45 U, SW46 J, SW47 M, SW48 Spacebar, SW49 F8, SW5 Left Shift, SW50 8, SW51 I, SW52 K, SW53 ,, SW54 F9, SW55 9, SW56 O, SW57 L, SW58 ., SW59 F10, SW60 0, SW61 P, SW62 ;, SW63 /, SW64 F11, SW65 -, SW66 [, SW67 ', SW69 F12, SW70 =, SW71 ], SW74 prntsrc, SW75 backspace, SW76 \, SW78 SHIFT, SW79 del, SW8 Esc, SW80 opt, SW82 ENTER, SW83 up, SW84 fn, SW85 pgup, SW86 pgdn, SW87 home, SW88 end, SW89 Control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

Commit message: July 26 update
Parts:
- removed SW1: EC11E15244G1, 2026-07-22_12-53-14:EC11E15244G1_AAL, symbol 2026-07-22_12-53-14:EC11E15244G1
- added H1, H2, H3, H4, H5, H6, H7, H8: MountingHole, MountingHole:MountingHole_2.5mm, symbol Mechanical:MountingHole
- added SW6: RotaryEncoder_Switch_MP, Rotary_Encoder:RotaryEncoder_Alps_EC11E-Switch_Vertical_H20mm, symbol Device:RotaryEncoder_Switch_MP
Connections:
- net A: now also SW6.A
- net B: now also SW6.C
- net C: now also SW6.S1
- net GND: now also SW6.B, SW6.S2

Commit message: Added production files
Parts:
- SW10, SW11, SW12, SW13, SW14, SW15, SW16, SW17, SW18, SW19, SW2, SW20, SW21, SW22, SW23, SW24, SW25, SW26, SW27, SW28, SW29, SW30, SW31, SW32, SW33, SW34, SW35, SW36, SW37, SW38, SW39, SW4, SW40, SW41, SW42, SW43, SW44, SW45, SW46, SW47, SW48, SW49, SW5, SW50, SW51, SW52, SW53, SW54, SW55, SW56, SW57, SW58, SW59, SW60, SW61, SW62, SW63, SW64, SW65, SW66, SW67, SW69, SW70, SW71, SW74, SW75, SW76, SW78, SW79, SW8, SW80, SW82, SW83, SW84, SW85, SW86, SW87, SW88, SW89, SW9, SW90, SW91, SW92: now left out of the parts list

Commit message: keyey
Parts:
- removed H5, H7: MountingHole, MountingHole:MountingHole_2.5mm, symbol Mechanical:MountingHole
