File: Keyey/LED.kicad_sch (KiCad schematic)
At the start: 170 parts

Commit message: July 26 update
Connections:
- net GND: no longer D165.4 (DOUT), D166.2 (DIN)
- new net: D165.4 (DOUT), D166.2 (DIN)
Changed lines of the file:
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@@
 	)
 	(junction
-		(at 26.67 218.44)
-		(diameter 0)
-		(color 0 0 0 0)
-	)
-	(junction
 		(at 80.01 96.52)
 		(diameter 0)
@@
 	(wire
 		(pts
-			(xy 26.67 215.9) (xy 26.67 218.44)
+			(xy 26.67 215.9) (xy 26.67 226.06)
 		)
 		(stroke
@@
 	(wire
 		(pts
-			(xy 26.67 218.44) (xy 26.67 226.06)
-		)
-		(stroke
-			(width 0)
-			(type default)
-		)
-	)
-	(wire
-		(pts
 			(xy 179.07 71.12) (xy 26.67 71.12)
 		)
@@
 		(in_pos_files yes)
 		(dnp no)
-		(fields_autoplaced yes)
 		(property "Reference" "#PWR0283"
 			(at 38.1 218.44 0)
@@
 		)
 		(property "Value" "+5V"
-			(at 30.48 218.4399 90)
+			(at 32.512 216.662 90)
 			(show_name no)
 			(do_not_autoplace no)
@@
 					(unit 1)
 				)
-			)
-		)
-	)
-	(symbol
-		(lib_id "power:GND")
-		(at 26.67 218.44 90)
-		(unit 1)
-		(body_style 1)
-		(exclude_from_sim no)
-		(in_bom yes)
-		(on_board yes)
-		(in_pos_files yes)
-		(dnp no)
-		(fields_autoplaced yes)
-		(property "Reference" "#PWR0282"
-			(at 33.02 218.44 0)
-			(hide yes)
-			(show_name no)
-			(do_not_autoplace no)
-			(effects
-				(font
-					(size 1.27 1.27)
-				)
-			)
-		)
-		(property "Value" "GND"
-			(at 30.48 218.4399 90)
-			(show_name no)
-			(do_not_autoplace no)
-			(effects
-				(font
-					(size 1.27 1.27)
-				)
-				(justify right)
-			)
-		)
-		(property "Footprint" ""
-			(at 26.67 218.44 0)
-			(hide yes)
-			(show_name no)
-			(do_not_autoplace no)
-			(effects
-				(font
-					(size 1.27 1.27)
-				)
-			)
-		)
-		(property "Datasheet" ""
-			(at 26.67 218.44 0)
-			(hide yes)
-			(show_name no)
-			(do_not_autoplace no)
-			(effects
-				(font
-					(size 1.27 1.27)
-				)
-			)
-		)
-		(property "Description" "Power symbol creates a global label with name \"GND\" , ground"
-			(at 26.67 218.44 0)
-			(hide yes)
-			(show_name no)
-			(do_not_autoplace no)
-			(effects
-				(font
-					(size 1.27 1.27)
-				)
-			)
-		)
-		(pin "1"
-		)
-		(instances
-			(project "Keyey"
-				(path "/edd52eb0-3b06-40db-996c-6985879c755e/bca6c043-d1b0-40dc-a0ac-a65731fd1828"
-					(reference "#PWR0282")
-					(unit 1)
-				)
